File: rfduino-lure/$rfduino-lure.sch (KiCad schematic (older format))
At the start: 4 parts, among them U1 RFDUINO_SHEILD, U2 MAX_LSE, U3 RFDUINO_IO

Commit message: some refactoring
Parts:
- removed U1: RFDUINO_SHEILD, ~, symbol RFDUINO_SHEILD
- removed U3: RFDUINO_IO, symbol RFDUINO_IO
- added U1: RFDUINO_IO, ~, symbol RFDUINO_IO
- added USB1: USB-PROGRAMMER, ~, symbol USB-PROGRAMMER
Connections:
- net at BLE1.1: now also U1.1 (GND)
- net at BLE1.12 (GND), U2.2 (GND): now also USB1.1 (GND)
- net at BLE1.13 (+3V), U2.4 (3V3): now also USB1.2 (+3V)
- net at BLE1.14 (RESET): now also USB1.3 (RESET)
- net at BLE1.15 (FACTORY): now also USB1.4 (FACTORY)
- net at BLE1.16 (GPIO_0/AREF), U2.17 (GPIO_UART2_TXD): now also USB1.5 (GPIO_0/AREF)
- net at BLE1.17 (GPIO_1), U2.19 (GPIO_UART2_RXD): now also USB1.6 (GPIO_1)
- net at BLE1.2 (GND): now also U1.2 (GND)
- net at BLE1.3 (GPIO_2): now also U1.3 (GPIO_2)
- net at BLE1.4 (GPIO_3): now also U1.4 (GPIO_3)
- net at BLE1.5 (GPIO_4): now also U1.5 (GPIO_4)
- net at BLE1.6 (GPIO_5): now also U1.6 (GPIO_5)
- net at BLE1.7 (GPIO_6): now also U1.7 (GPIO_6)
- net at BLE1.8 (GND): now also U1.8 (GND)
Changed lines of the file:
@@
 Sheet 1 1
 Title ""
-Date "27 mar 2015"
+Date "28 mar 2015"
 Rev ""
 Comp ""
@@
 	-1   0    0    1
 $EndComp
-$Comp
-L RFDUINO_IO U3
-U 1 1 551519C4
-P 4100 3000
-F 0 "U3" H 4100 3000 60  0000 C CNN
-F 1 "RFDUINO_IO" H 4100 4050 60  0000 C CNN
-F 2 "" H 4100 3000 60  0000 C CNN
-F 3 "" H 4100 3000 60  0000 C CNN
-	1    4100 3000
-	1    0    0    -1
-$EndComp
-$Comp
-L RFDUINO_SHEILD U1
-U 1 1 55152170
-P 3300 3900
-F 0 "U1" H 3300 3900 60  0000 C CNN
-F 1 "RFDUINO_SHEILD" H 3300 4950 60  0000 C CNN
-F 2 "~" H 3300 3900 60  0000 C CNN
-F 3 "~" H 3300 3900 60  0000 C CNN
-	1    3300 3900
-	0    -1   -1   0
-$EndComp
 Wire Wire Line
 	1200 4600 1200 7600
@@
 Connection ~ 1200 6450
 Wire Wire Line
-	3700 2200 1100 2200
-Wire Wire Line
-	1100 2200 1100 3050
-Wire Wire Line
 	1200 3050 1200 2300
-Wire Wire Line
-	1200 2300 3700 2300
 Wire Wire Line
 	1300 3050 1300 2400
 Wire Wire Line
-	1300 2400 3700 2400
-Wire Wire Line
 	1400 3050 1400 2500
-Wire Wire Line
-	1400 2500 3700 2500
-Wire Wire Line
-	3700 2600 1500 2600
 Wire Wire Line
 	1500 2600 1500 3050
 Wire Wire Line
 	1600 3050 1600 2700
-Wire Wire Line
-	1600 2700 3700 2700
-Wire Wire Line
-	3700 2800 1700 2800
-Wire Wire Line
-	1700 2800 1700 3050
-Wire Wire Line
-	1800 3050 1800 2900
-Wire Wire Line
-	1800 2900 3700 2900
-Wire Wire Line
-	2550 3100 2550 2300
-Connection ~ 2550 2300
-Wire Wire Line
-	2650 3100 2650 2400
-Connection ~ 2650 2400
-Wire Wire Line
-	2750 3100 2750 2500
-Connection ~ 2750 2500
-Wire Wire Line
-	2850 3100 2850 2600
-Connection ~ 2850 2600
-Wire Wire Line
-	2950 3100 2950 2700
-Connection ~ 2950 2700
 Wire Wire Line
 	2850 4600 2850 4950
@@
 Wire Wire Line
 	2450 6300 1100 6300
+$Comp
+L USB-PROGRAMMER USB1
+U 1 1 55163475
+P 2600 4200
+F 0 "USB1" H 2650 3650 60  0000 C CNN
+F 1 "USB-PROGRAMMER" H 2600 4500 60  0000 C CNN
+F 2 "~" H 2600 4200 60  0000 C CNN
+F 3 "~" H 2600 4200 60  0000 C CNN
+	1    2600 4200
+	0    -1   -1   0
+$EndComp
+$Comp
+L RFDUINO_IO U1
+U 1 1 5516349D
+P 2950 3000
+F 0 "U1" H 2950 3000 60  0000 C CNN
+F 1 "RFDUINO_IO" H 2950 4050 60  0000 C CNN
+F 2 "~" H 2950 3000 60  0000 C CNN
+F 3 "~" H 2950 3000 60  0000 C CNN
+	1    2950 3000
+	1    0    0    -1
+$EndComp
+Wire Wire Line
+	1600 2700 2550 2700
+Wire Wire Line
+	2550 2800 1700 2800
+Wire Wire Line
+	1700 2800 1700 3050
+Wire Wire Line
+	2550 2900 1800 2900
+Wire Wire Line
+	1800 2900 1800 3050
+Wire Wire Line
+	1100 3050 1100 2200
+Wire Wire Line
+	1100 2200 2550 2200
+Wire Wire Line
+	1400 2500 2550 2500
+Wire Wire Line
+	2550 2600 1500 2600
+Wire Wire Line
+	1300 2400 2550 2400
+Wire Wire Line
+	1200 2300 2550 2300
 $EndSCHEMATC
